File: kicad-proj/ina3221-mcu.kicad_pcb (KiCad board)
At the start: 2 copper layers, 57 x 44 mm, 45 parts, among them J1 Conn_01x08_Pin, J11 BAT_O_0P, J13 BAT_O_1P, J16 20Vin, J2 GND, J3 BAT0P, J4 BAT_O_0P, J7 BAT0P, J9 BAT1P, SW1 SW_Push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

Commit message: first release
Parts:
- removed C4, C5: 10uF, Capacitor_SMD:C_0603_1608Metric_Pad1.08x0.95mm_HandSolder
- removed C6, C7, C8: 2.2uF, Capacitor_SMD:C_0603_1608Metric_Pad1.08x0.95mm_HandSolder
- removed J1: Conn_01x08_Pin, Connector_PinHeader_1.00mm:PinHeader_1x08_P1.00mm_Vertical
- removed RN1, RN2: 4.7K, Resistor_SMD:R_Array_Concave_4x0603
- removed SW2, SW3: SW_Push, Button_Switch_SMD:SW_SPST_TL3305A
- removed TP1, TP2: TestPoint, TestPoint:TestPoint_Pad_1.0x1.0mm
- removed TP3: SWCLK, TestPoint:TestPoint_Pad_2.0x2.0mm
- removed TP4: SWDIO, TestPoint:TestPoint_Pad_2.0x2.0mm
- removed TP7: ~, TestPoint:TestPoint_Pad_1.0x1.0mm
- added R12: 10K, Resistor_SMD:R_0603_1608Metric_Pad0.98x0.95mm_HandSolder, F.Cu at (27.3, 50.8)
- added R13: 10K, Resistor_SMD:R_0603_1608Metric_Pad0.98x0.95mm_HandSolder, F.Cu at (27.3, 52.8)
- DS1: value OLED-128O064D -> 12864-21M; footprint Display:OLED-128O064D -> Display:AG12864E; moved to B.Cu
- J11, J13, J3, J4, J7, J9: moved to F.Cu
- R1, R2: value 0.05 -> 0.02
- R10: value 0.04 -> 0.02
- R7: value 910K -> 330
- R8: value 4.7K -> 10K
- moved J16 61.8 mm to (19.6, 71.4), turned to 180 degrees
- moved U4 61.4 mm to (29.4, 69.7), turned to 180 degrees
- moved U3 60.3 mm to (24.4, 69.7), turned to 180 degrees
- moved C3 57.9 mm to (32.8, 69.9), turned to -90 degrees
- moved J2 56.2 mm to (19.5, 67.5), turned to 180 degrees
- moved R7 56.1 mm to (29.8, 74.0), turned to 180 degrees
- moved R8 55.4 mm to (30.2, 66.6), turned to 180 degrees
- moved J3 54.8 mm to (19.6, 61.3)
- moved J4 53.8 mm to (19.6, 53.6)
- moved R10 52.5 mm to (19.6, 57.5), turned to 90 degrees
- moved C9 51.5 mm to (29.8, 62.0), turned to 180 degrees
- moved DS1 48.1 mm to (37.5, 75.3), turned to 0 degrees
- moved R9 47.6 mm to (22.4, 61.1), turned to -90 degrees
- moved R11 46.7 mm to (22.4, 54.0), turned to 90 degrees
- moved C10 44.5 mm to (22.4, 57.5), turned to 90 degrees
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Connections:
- C3 pad 1: 5v0 -> 3v3
- C9 pad 2: Net-(DS1-~{RES}) -> Net-(U2-NRST)
- DS1 pad 1: GND -> 5v0
- DS1 pad 10: Net-(DS1-BS0) -> unconnected-(DS1-DB3-Pad10)
- DS1 pad 11: GND -> unconnected-(DS1-DB4-Pad11)
- DS1 pad 12: GND -> unconnected-(DS1-DB5-Pad12)
- DS1 pad 13: Net-(DS1-~{CS}) -> unconnected-(DS1-DB6-Pad13)
- DS1 pad 14: Net-(DS1-~{RES}) -> unconnected-(DS1-DB7-Pad14)
- DS1 pad 16: GND -> unconnected-(DS1-NC-Pad16)
- DS1 pad 17: GND -> unconnected-(DS1-~{RST}-Pad17)
- DS1 pad 18: Net-(DS1-D0) -> unconnected-(DS1-Vout-Pad18)
- DS1 pad 19: Net-(DS1-D1) -> Net-(DS1-LEDA/EL)
- DS1 pad 2: Net-(DS1-C2N) -> GND
- DS1 pad 20: unconnected-(DS1-D2-Pad20) -> GND
- DS1 pad 3: Net-(DS1-C2P) -> Net-(DS1-RS)
- DS1 pad 4: Net-(DS1-C1P) -> Net-(DS1-RS)
- DS1 pad 5: Net-(DS1-C1N) -> Net-(DS1-R/~{W})
- DS1 pad 6: 3v3 -> Net-(DS1-E)
- DS1 pad 8: GND -> unconnected-(DS1-DB1-Pad8)
- DS1 pad 9: 3v3 -> unconnected-(DS1-DB2-Pad9)
- R7 pad 1: Net-(DS1-IREF) -> Net-(DS1-LEDA/EL)
- R7 pad 2: GND -> 5v0
- R8 pad 1: Net-(DS1-BS0) -> Net-(DS1-RS)
- SW1 pad 1: GND -> Net-(U2-NRST)
- SW1 pad 2: SWCLK -> GND
- U1 pad 4: 5v0 -> 3v3
- U1 pad 6: SCL2 -> SCL1
- U1 pad 7: SDA2 -> SDA1
- U2 pad 10: SCL3 -> unconnected-(U2-PA3-Pad10)
- U2 pad 11: Net-(DS1-~{CS}) -> unconnected-(U2-PA4-Pad11)
- U2 pad 12: Net-(DS1-D0) -> Net-(DS1-R/~{W})
- U2 pad 13: Net-(U2-PA6) -> unconnected-(U2-PA6-Pad13)
- U2 pad 14: Net-(DS1-D1) -> Net-(DS1-E)
- U2 pad 15: Net-(U2-PB0/PB1/PB2/PA8) -> unconnected-(U2-PB0/PB1/PB2/PA8-Pad15)
- U2 pad 16: SCL2 -> unconnected-(U2-PA11/PA9-Pad16)
- U2 pad 17: SDA2 -> unconnected-(U2-PA12/PA10-Pad17)
- U2 pad 20: Net-(U2-PB3/PB4/PB5/PB6) -> unconnected-(U2-PB3/PB4/PB5/PB6-Pad20)
- U2 pad 3: Net-(U2-PC15) -> unconnected-(U2-PC15-Pad3)
- U2 pad 6: Net-(DS1-~{RES}) -> Net-(U2-NRST)
- U2 pad 7: SDA4 -> unconnected-(U2-PA0-Pad7)
- U2 pad 8: SCL4 -> unconnected-(U2-PA1-Pad8)
- U2 pad 9: SDA3 -> unconnected-(U2-PA2-Pad9)
Routing:
- net SWCLK: track 64.6 -> 0.00 mm, vias 3 -> 0
- net Net-(DS1-LEDA/EL): track 0.00 -> 54.7 mm
- net SWDIO: track 54.3 -> 0.00 mm, vias 3 -> 0
- net Net-(U2-NRST): track 0.00 -> 37.5 mm
- net Net-(U2-PC15): track 36.6 -> 0.00 mm, vias 2 -> 0
- net GND: track 191.8 -> 155.3 mm, vias 1 -> 0
- net 3v3: track 50.8 -> 29.6 mm
- net Net-(DS1-~{RES}): track 19.2 -> 0.00 mm, vias 2 -> 0
- net SDA2: track 17.2 -> 0.00 mm, vias 2 -> 0
- net SCL2: track 17.0 -> 0.00 mm, vias 2 -> 0
- net Net-(DS1-D1): track 16.5 -> 0.00 mm
- net Net-(DS1-D0): track 15.0 -> 0.00 mm
- net Net-(U1-IN-1): track 3.46 -> 16.0 mm
- net Net-(DS1-~{CS}): track 11.2 -> 0.00 mm
- net Net-(DS1-RS): track 0.00 -> 9.34 mm
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Other:
- board outline removed
