File: kicad-proj/ina3221-mcu.kicad_sch (KiCad schematic)
At the start: 45 parts, among them J1 Conn_01x08_Pin, J11 BAT_O_0P, J13 BAT_O_1P, J16 20Vin, J2 GND, J3 BAT0P, J4 BAT_O_0P, J7 BAT0P, J9 BAT1P, SW1 SW_Push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

Commit message: first release
Parts:
- removed C4, C5: 10uF, Capacitor_SMD:C_0603_1608Metric_Pad1.08x0.95mm_HandSolder, symbol Device:C
- removed C6, C7, C8: 2.2uF, Capacitor_SMD:C_0603_1608Metric_Pad1.08x0.95mm_HandSolder, symbol Device:C
- removed DS1: OLED-128O064D, Display:OLED-128O064D, symbol Display_Graphic:OLED-128O064D
- removed J1: Conn_01x08_Pin, Connector_PinHeader_1.00mm:PinHeader_1x08_P1.00mm_Vertical, symbol Connector:Conn_01x08_Pin
- removed RN1, RN2: 4.7K, Resistor_SMD:R_Array_Concave_4x0603, symbol Device:R_Pack04
- removed SW1, SW2: SW_Push, Button_Switch_SMD:SW_SPST_TL3305A, symbol Switch:SW_Push
- removed TP1, TP2: TestPoint, TestPoint:TestPoint_Pad_1.0x1.0mm, symbol Connector:TestPoint
- removed TP3: SWCLK, TestPoint:TestPoint_Pad_2.0x2.0mm, symbol Connector:TestPoint
- removed TP4: SWDIO, TestPoint:TestPoint_Pad_2.0x2.0mm, symbol Connector:TestPoint
- removed TP7: ~, TestPoint:TestPoint_Pad_1.0x1.0mm, symbol Connector:TestPoint
- added DS1: 12864-21M, Display:AG12864E, symbol Display_Graphic:AG12864E
- added R12, R13: 10K, Resistor_SMD:R_0603_1608Metric_Pad0.98x0.95mm_HandSolder, symbol Device:R
- R1, R2: value 0.05 -> 0.02
- R10: value 0.04 -> 0.02
- R7: value 910K -> 330
- R8: value 4.7K -> 10K
- renumbered SW3 to SW1
Connections:
- net 3v3: now also C3.1, U1.4 (VS), R12.2, R13.2
- net 5v0: now also R7.2, DS1.1 (VCC); no longer C3.1, U1.4 (VS)
- net GND: now also DS1.15 (PSB), DS1.2 (GND), DS1.20 (LEDK/EL); no longer R7.2
- net SCL1: now also U1.6 (SCL), R12.1
- net SDA1: now also U1.7 (SDA), R13.1
- net at R8.1: now also DS1.3 (VO), DS1.4 (RS)
- net at SW1.1: now also C9.2, U2.6 (NRST); no longer U2.3 (PC15)
- net at U2.12 (PA5): now also DS1.5 (R/~{W})
- net at U2.14 (PA7): now also DS1.6 (E)
- net at R7.1: now also DS1.19 (LEDA/EL)
- net SCL2: no longer names the net of U2.16 (PA11/PA9)
- net SCL2: no longer U1.6 (SCL)
- net SCL3: no longer names the net of U2.10 (PA3)
- net SCL4: no longer names the net of U2.8 (PA1)
- net SDA2: no longer names the net of U2.17 (PA12/PA10)
- net SDA2: no longer U1.7 (SDA)
- net SDA3: no longer names the net of U2.9 (PA2)
- net SDA4: no longer names the net of U2.7 (PA0)
- no-connect marks 6 -> 27
Other:
- note added: "spi_clk"
- note added: "spi_mosi"
